File: KiCad_projekti/Elektroniikkapaja.kicad_sch (KiCad schematic)
At the start: 2 parts, among them U1 ATmega644-20A

Commit message: testaus onko oikea versio
Parts:
- removed R1: 10k, Resistor_SMD:R_0805_2012Metric, symbol Device:R
- added C? (x14): C, symbol Device:C
- added D?: D_Zener, symbol Device:D_Zener
- added J?: Conn_01x06_Pin, Connector_PinHeader_2.54mm:PinHeader_1x06_P2.54mm_Vertical, symbol Connector:Conn_01x06_Pin
- added J?: Conn_Coaxial, symbol Connector:Conn_Coaxial
- added L? (x3): L, symbol Device:L
- added R? (x6): R, symbol Device:R
- added R?: 10k, Resistor_SMD:R_0805_2012Metric_Pad1.20x1.40mm_HandSolder, symbol Device:R
- added U2: ~, symbol Weather-station-project-imported-compnents:SPV1040
- added U?: ~, symbol Weather-station-project-imported-compnents:Micrf113
- added U?: MCP1700x-330xxTO, Package_TO_SOT_THT:TO-92_Inline, symbol Regulator_Linear:MCP1700x-330xxTO
- added Y? (x2): Crystal, symbol Device:Crystal
Connections:
- net GND: now also U1.18 (GND), U1.28 (GND), U1.39 (GND), U1.6 (GND), C?.1, C?.1, C?.1, C?.2, C?.2, C?.2, C?.2, C?.2, C?.2, C?.2, C?.2, C?.2, D?.2 (A), J?.2 (Ext), R?.1, U2.2 (GND), U?.1 (GND), U?.2 (VSS)
- net +3.3VDc: now reaches U1.17 (VCC), U1.38 (VCC), U1.5 (VCC)
- net +3.3VDc: now also C?.1, C?.1, L?.1, R?.1, U?.3 (VDD), U?.3 (VO)
- net at U1.4 (~{RESET}): now also R?.2
- net at U1.7 (XTAL2): now also C?.2, Y?.1
- net at U1.8 (XTAL1): now also C?.2, Y?.2
- net Vcc: no longer names the net of U1.33 (PA4)
- new net: C?.1, R?.1, U2.1 (MPP-SET), U2.8 (XSHUT)
- new net: L?.2, U2.3 (Lx)
- new net: C?.2, R?.1, R?.2, U2.4 (VOUT)
- new net: C?.1, R?.1, R?.2, U2.5 (VCTRL)
- new net: C?.2, R?.1, U2.6 (ICTRL-)
- new net: C?.1, R?.1, U2.7 (ICTRL+)
- new net: C?.1, L?.2
- new net: C?.2, L?.2, U?.1 (PAOUT)
- new net: C?.1, J?.1 (In), L?.1
- new net: C?.1, U?.4 (XTLOUT), Y?.1
- new net: C?.1, U?.5 (XTLIN), Y?.2
- new net ASK: U?.6 (ASK)
- new net LiPo_Battery: C?.1, D?.1 (K), R?.2, R?.2, R?.2, U?.2 (VI)
- new net Solar_panel: C?.1, L?.1, R?.2
Other:
- note added: "ASK Radio transmitter"
- note added: "ICSP header"
- note added: "PMIC"
- note added: "Sensors"
- moved on the sheet: U1
