File: KiCad_projekti/Elektroniikkapaja-lähetin/Elektroniikkapaja.kicad_pcb (KiCad board)
At the start: 2 copper layers, 2 parts, among them U1 ATmega644-20A

Commit message: nyt on valmista levyä
Parts:
- added BT1: Battery_Cell, Battery:BatteryHolder_MPD_BH-18650-PC2, F.Cu at (197.8, 143.5)
- added C1: 22pF, Capacitor_SMD:C_0805_2012Metric_Pad1.18x1.45mm_HandSolder, F.Cu at (253.7, 100.8)
- added C10: 100nF, Capacitor_SMD:C_0805_2012Metric_Pad1.18x1.45mm_HandSolder, F.Cu at (231.4, 80.8)
- added C11: 1uF, Capacitor_SMD:C_0805_2012Metric_Pad1.18x1.45mm_HandSolder, F.Cu at (240.8, 120.1)
- added C12: 1uF, Capacitor_SMD:C_0805_2012Metric_Pad1.18x1.45mm_HandSolder, F.Cu at (245.4, 120.1)
- added C13: 10uF, Capacitor_SMD:C_0805_2012Metric_Pad1.18x1.45mm_HandSolder, F.Cu at (223.0, 142.2)
- added C14: 1nF, Capacitor_SMD:C_0805_2012Metric_Pad1.18x1.45mm_HandSolder, F.Cu at (223.0, 133.6)
- added C15: 1uF, Capacitor_SMD:C_0805_2012Metric_Pad1.18x1.45mm_HandSolder, F.Cu at (234.7, 138.1)
- added C16: 1nF, Capacitor_SMD:C_0805_2012Metric_Pad1.18x1.45mm_HandSolder, F.Cu at (231.4, 142.3)
- added C17: 100nF, Capacitor_SMD:C_0805_2012Metric_Pad1.18x1.45mm_HandSolder, F.Cu at (217.2, 85.3)
- added C18: 4.7uF, Capacitor_SMD:C_1206_3216Metric_Pad1.33x1.80mm_HandSolder, F.Cu at (241.5, 127.1)
- added C19: 4.7uF, Capacitor_SMD:C_1206_3216Metric_Pad1.33x1.80mm_HandSolder, F.Cu at (228.5, 128.2)
- added C2: 22pF, Capacitor_SMD:C_0805_2012Metric_Pad1.18x1.45mm_HandSolder, F.Cu at (237.2, 100.8)
- added C20: 10uF, Capacitor_SMD:C_0805_2012Metric_Pad1.18x1.45mm_HandSolder, F.Cu at (238.0, 133.6)
- added C21: 100nF, Capacitor_SMD:C_0805_2012Metric_Pad1.18x1.45mm_HandSolder, F.Cu at (254.0, 90.9)
- added C22: 100nF, Capacitor_SMD:C_0805_2012Metric_Pad1.18x1.45mm_HandSolder, F.Cu at (226.9, 104.8)
- added C3: 4.7pF, Capacitor_SMD:C_0805_2012Metric_Pad1.18x1.45mm_HandSolder, F.Cu at (226.8, 77.5)
- added C4: 100nF, Capacitor_SMD:C_0805_2012Metric_Pad1.18x1.45mm_HandSolder, F.Cu at (237.2, 92.4)
- added C5: 10pF, Capacitor_SMD:C_0805_2012Metric_Pad1.18x1.45mm_HandSolder, F.Cu at (224.3, 81.5)
- added C6: 10uF, Capacitor_SMD:C_0805_2012Metric_Pad1.18x1.45mm_HandSolder, F.Cu at (237.2, 88.4)
- added C7: 10uF, Capacitor_SMD:C_0805_2012Metric_Pad1.18x1.45mm_HandSolder, F.Cu at (217.0, 87.9)
- added C8: 18pF, Capacitor_SMD:C_0805_2012Metric_Pad1.18x1.45mm_HandSolder, F.Cu at (217.0, 91.4)
- added C9: 18pF, Capacitor_SMD:C_0805_2012Metric_Pad1.18x1.45mm_HandSolder, F.Cu at (221.4, 91.4)
- added D1: LED, LED_SMD:LED_0805_2012Metric_Pad1.15x1.40mm_HandSolder, F.Cu at (233.9, 100.8)
- added D2: 5.1V Zener, Diode_THT:D_DO-35_SOD27_P7.62mm_Horizontal, F.Cu at (244.6, 135.9)
- added D3: LED, LED_SMD:LED_0805_2012Metric_Pad1.15x1.40mm_HandSolder, F.Cu at (238.0, 124.1)
- added D4: 1N4148, Diode_THT:D_DO-35_SOD27_P7.62mm_Horizontal, F.Cu at (233.1, 121.6)
- added H1: MountingHole, MountingHole:MountingHole_2.2mm_M2, F.Cu at (184.1, 74.3)
- added H2: MountingHole, MountingHole:MountingHole_2.2mm_M2, F.Cu at (250.8, 74.3)
- added H3: MountingHole, MountingHole:MountingHole_2.2mm_M2, F.Cu at (184.2, 140.8)
- added H4: MountingHole, MountingHole:MountingHole_2.2mm_M2, F.Cu at (250.9, 140.7)
- added J1: Conn_Coaxial, Connector_Coaxial:SMA_Amphenol_901-143_Horizontal, F.Cu at (217.4, 74.5)
- added J3: Conn_01x06_Pin, Connector_PinHeader_2.54mm:PinHeader_1x06_P2.54mm_Vertical, F.Cu at (231.4, 72.9)
- added J4: Conn_01x04_Pin, Connector_PinHeader_2.54mm:PinHeader_1x04_P2.54mm_Vertical, F.Cu at (251.7, 113.3)
- added J5: Conn_01x07_Socket, Connector_PinSocket_2.54mm:PinSocket_1x07_P2.54mm_Vertical, F.Cu at (214.5, 107.7)
- added J6: Conn_01x02_Pin, Connector_PinHeader_2.54mm:PinHeader_1x02_P2.54mm_Vertical, F.Cu at (231.4, 133.1)
- added J7: Conn_01x08_Pin, Connector_PinHeader_2.54mm:PinHeader_1x08_P2.54mm_Vertical, F.Cu at (184.2, 101.1)
- added J8: Solar_panel_connector, Connector_PinHeader_2.54mm:PinHeader_1x02_P2.54mm_Vertical, F.Cu at (183.6, 127.6)
- added J9: AVR-ISP-6, Connector_PinHeader_2.54mm:PinHeader_2x03_P2.54mm_Vertical, F.Cu at (235.6, 81.4)
- added L1: 82nH, Inductor_SMD:L_0805_2012Metric_Pad1.15x1.40mm_HandSolder, F.Cu at (224.3, 77.5)
- added L2: 470nF, Inductor_SMD:L_0805_2012Metric_Pad1.15x1.40mm_HandSolder, F.Cu at (220.7, 82.5)
- added L3: 10uH, inductor_footprint:WE-PD2_1054, F.Cu at (215.6, 138.2)
- added Q1: SSM3J371R, Package_TO_SOT_SMD:SOT-23-3, F.Cu at (233.5, 92.6)
- added Q2: SSM3J371R, Package_TO_SOT_SMD:SOT-23-3, F.Cu at (236.2, 109.5)
- added R10: 2k2, Resistor_SMD:R_0805_2012Metric_Pad1.20x1.40mm_HandSolder, F.Cu at (237.2, 96.5)
- added R11: R, Resistor_SMD:R_0805_2012Metric_Pad1.20x1.40mm_HandSolder, F.Cu at (233.9, 88.4)
- added R12: R_Photo, Resistor_THT:R_Axial_DIN0204_L3.6mm_D1.6mm_P2.54mm_Vertical, F.Cu at (230.6, 87.2)
- added R13: 150k, Resistor_SMD:R_0805_2012Metric_Pad1.20x1.40mm_HandSolder, F.Cu at (231.1, 103.1)
- added R14: 300k, Resistor_SMD:R_0805_2012Metric_Pad1.20x1.40mm_HandSolder, F.Cu at (233.9, 105.2)
- added R15: 330r, Resistor_SMD:R_0805_2012Metric_Pad1.20x1.40mm_HandSolder, F.Cu at (233.6, 124.1)
- added R16: 4k7, Resistor_SMD:R_0805_2012Metric_Pad1.20x1.40mm_HandSolder, F.Cu at (236.7, 127.2)
- added R17: 2k2, Resistor_SMD:R_0805_2012Metric_Pad1.20x1.40mm_HandSolder, F.Cu at (237.2, 105.2)
- added R18: 4k7, Resistor_SMD:R_0805_2012Metric_Pad1.20x1.40mm_HandSolder, F.Cu at (218.7, 109.2)
- added R19: 4k7, Resistor_SMD:R_0805_2012Metric_Pad1.20x1.40mm_HandSolder, F.Cu at (218.7, 114.5)
- added R2: 150r, Resistor_SMD:R_0805_2012Metric_Pad1.20x1.40mm_HandSolder, F.Cu at (233.9, 96.5)
- added R20: 4k7, Resistor_SMD:R_0805_2012Metric_Pad1.20x1.40mm_HandSolder, F.Cu at (218.7, 119.6)
- added R21: 4k7, Resistor_SMD:R_0805_2012Metric_Pad1.20x1.40mm_HandSolder, F.Cu at (223.9, 126.4)
- added R3: 1k, Resistor_SMD:R_0805_2012Metric_Pad1.20x1.40mm_HandSolder, F.Cu at (223.0, 137.9)
- added R4: 4k7, Resistor_SMD:R_0805_2012Metric_Pad1.20x1.40mm_HandSolder, F.Cu at (247.4, 80.8)
- added R5: 1k, Resistor_SMD:R_0805_2012Metric_Pad1.20x1.40mm_HandSolder, F.Cu at (238.0, 138.2)
- added R6: 1k, Resistor_SMD:R_0805_2012Metric_Pad1.20x1.40mm_HandSolder, F.Cu at (241.3, 138.2)
- added R7: 680mohm, Resistor_SMD:R_0805_2012Metric_Pad1.20x1.40mm_HandSolder, F.Cu at (241.3, 133.6)
- added R8: 160k, Resistor_SMD:R_0805_2012Metric_Pad1.20x1.40mm_HandSolder, F.Cu at (234.7, 142.2)
- added R9: 68k, Resistor_SMD:R_0805_2012Metric_Pad1.20x1.40mm_HandSolder, F.Cu at (238.0, 142.2)
- added SW1: SW_SPDT, Button_Switch_THT:SW_CuK_JS202011CQN_DPDT_Straight, F.Cu at (249.2, 132.3)
- added SW_reset1: SW_Push, Button_Switch_SMD:SW_SPST_TL3305A, F.Cu at (244.3, 108.7)
- added U2: ~, Package_SO:TSSOP-8_4.4x3mm_P0.65mm, F.Cu at (228.5, 138.0)
- added U3: Micrf113, Package_TO_SOT_SMD:SOT-23-6_Handsoldering, F.Cu at (221.7, 86.8)
- added U4: MCP1700x-330xxTO, Package_TO_SOT_THT:TO-92_Inline, F.Cu at (241.8, 116.7)
- added U5: DS18S20, Package_TO_SOT_THT:TO-92_Inline, F.Cu at (252.0, 79.8)
- added U6: MCP73831-2-OT, Package_TO_SOT_SMD:SOT-23-5, F.Cu at (233.1, 127.3)
- added U7: SN74LS07N, Package_DIP:DIP-14_W7.62mm, F.Cu at (221.1, 107.7)
- added Y1: Crystal 16MHz, Crystal:Crystal_HC49-U_Vertical, F.Cu at (243.2, 101.8)
- added Y2: Crystal 13.56MHz, Crystal:Crystal_HC49-U_Vertical, F.Cu at (215.3, 96.8)
- R1: footprint Resistor_SMD:R_0805_2012Metric -> Resistor_SMD:R_0805_2012Metric_Pad1.20x1.40mm_HandSolder
- moved R1 139.8 mm to (251.5, 108.0), turned to 90 degrees
- moved U1 128.6 mm to (246.0, 91.3), turned to 90 degrees
Connections:
- R1 pad 1: Net-(U1-PB0) -> +3.3VDc
- R1 pad 2: GND -> RST
- U1 pad 1: unconnected-(U1-PB5-Pad1) -> MOSI
- U1 pad 10: unconnected-(U1-PD1-Pad10) -> Tx
- U1 pad 11: unconnected-(U1-PD2-Pad11) -> PD2
- U1 pad 12: unconnected-(U1-PD3-Pad12) -> PD3
- U1 pad 13: unconnected-(U1-PD4-Pad13) -> PD4
- U1 pad 17: Net-(U1-VCC-Pad17) -> +3.3VDc
- U1 pad 18: Net-(U1-GND-Pad18) -> GND
- U1 pad 19: unconnected-(U1-PC0-Pad19) -> SCL
- U1 pad 2: unconnected-(U1-PB6-Pad2) -> MISO
- U1 pad 20: unconnected-(U1-PC1-Pad20) -> SDA
- U1 pad 21: unconnected-(U1-PC2-Pad21) -> One_wire
- U1 pad 22: unconnected-(U1-PC3-Pad22) -> CS_BLVL
- U1 pad 27: unconnected-(U1-AVCC-Pad27) -> +3.3VDc
- U1 pad 28: Net-(U1-GND-Pad18) -> GND
- U1 pad 3: unconnected-(U1-PB7-Pad3) -> SCK
- U1 pad 32: unconnected-(U1-PA5-Pad32) -> PA5
- U1 pad 33: unconnected-(U1-PA4-Pad33) -> PA4
- U1 pad 36: unconnected-(U1-PA1-Pad36) -> LDR
- U1 pad 37: unconnected-(U1-PA0-Pad37) -> battery_lvl
- U1 pad 38: Net-(U1-VCC-Pad17) -> +3.3VDc
- U1 pad 39: Net-(U1-GND-Pad18) -> GND
- U1 pad 4: unconnected-(U1-~{RESET}-Pad4) -> RST
- U1 pad 40: Net-(U1-PB0) -> PB0
- U1 pad 41: unconnected-(U1-PB1-Pad41) -> CS_LDR
- U1 pad 42: unconnected-(U1-PB2-Pad42) -> CS_0
- U1 pad 43: unconnected-(U1-PB3-Pad43) -> int_led
- U1 pad 44: unconnected-(U1-PB4-Pad44) -> ASK
- U1 pad 5: Net-(U1-VCC-Pad17) -> +3.3VDc
- U1 pad 6: Net-(U1-GND-Pad18) -> GND
- U1 pad 7: unconnected-(U1-XTAL2-Pad7) -> Net-(U1-XTAL2)
- U1 pad 8: unconnected-(U1-XTAL1-Pad8) -> Net-(U1-XTAL1)
- U1 pad 9: unconnected-(U1-PD0-Pad9) -> Rx
Routing:
- net +3.3VDc: track 0.00 -> 256.9 mm, vias 0 -> 6
- net GND: track 0.00 -> 128.8 mm, vias 0 -> 128
- net PD4: track 0.00 -> 115.2 mm, vias 0 -> 1
- net PD3: track 0.00 -> 111.5 mm, vias 0 -> 1
- net PD2: track 0.00 -> 109.8 mm, vias 0 -> 1
- net LiPo_Battery: track 0.00 -> 94.5 mm
- net PA5: track 0.00 -> 83.2 mm, vias 0 -> 1
- net RST: track 0.00 -> 82.8 mm, vias 0 -> 4
- net PA4: track 0.00 -> 80.0 mm, vias 0 -> 1
- net PB0: track 0.00 -> 77.2 mm, vias 0 -> 1
- net CS_0: track 0.00 -> 57.9 mm, vias 0 -> 1
- net SCK_5V: track 0.00 -> 52.5 mm, vias 0 -> 1
- net MOSI: track 0.00 -> 50.2 mm, vias 0 -> 1
- net SCK: track 0.00 -> 50.1 mm, vias 0 -> 1
- net MOSI_5V: track 0.00 -> 47.6 mm, vias 0 -> 1
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- added copper zone on B.Cu, net GND
- added copper zone on F.Cu, net GND
- added copper zone on F.Cu, net Net-(U2-Lx)
Other:
- board outline added: 77 x 77 mm
- board text added: "+"
- board text added: "+3.3V"
- board text added: "+5Vin"
- board text added: "+Vin"
- board text added: "-"
- board text added: "2024"
- board text added: "3.3V"
- board text added: "BMP280"
- board text added: "CS"
- board text added: "ELEC-C8701"
- board text added: "GND"
- board text added: "ICSP"
- board text added: "PA4"
- board text added: "PA5"
- board text added: "PB0"
- board text added: "PD2"
- board text added: "PD3"
- board text added: "PD4"
- board text added: "Ryhmä 16"
- board text added: "SCK"
- board text added: "SCL"
- board text added: "SDA"
- board text added: "SDI"
- board text added: "SDO"
- board text added: "Solar panel"
- board text added: "Solar↔External"
- board text added: "UART"
- board text added: "Wireless Weather Station"
- board text added: "x"
