File: KiCad_projekti/Elektroniikkapaja-lähetin/Elektroniikkapaja.kicad_sch (KiCad schematic)
At the start: 59 parts, among them J1 Conn_Coaxial, J2 AVR-ISP-6, J3 Conn_01x06_Pin, J4 Conn_01x04_Pin, J5 Conn_01x06_Socket, J6 Conn_01x02_Pin, Q1 PMOS, SW1 SW_SPDT, U1 ATmega644-20A, U3 Micrf113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

Commit message: nyt on valmista levyä
Parts:
- removed J2: AVR-ISP-6, Connector_PinHeader_2.54mm:PinHeader_2x03_P2.54mm_Vertical, symbol Connector:AVR-ISP-6
- removed J5: Conn_01x06_Socket, Connector_PinHeader_2.54mm:PinHeader_1x06_P2.54mm_Vertical, symbol Connector:Conn_01x06_Socket
- added BT1: Battery_Cell, Battery:BatteryHolder_MPD_BH-18650-PC2, symbol Device:Battery_Cell
- added C21, C22: 100nF, Capacitor_SMD:C_0805_2012Metric_Pad1.18x1.45mm_HandSolder, symbol Device:C
- added D4: 1N4148, Diode_THT:D_DO-35_SOD27_P7.62mm_Horizontal, symbol Device:D
- added H1, H2, H3, H4: MountingHole, MountingHole:MountingHole_2.2mm_M2, symbol Mechanical:MountingHole
- added J5: Conn_01x07_Socket, Connector_PinSocket_2.54mm:PinSocket_1x07_P2.54mm_Vertical, symbol Connector:Conn_01x07_Socket
- added J7: Conn_01x08_Pin, Connector_PinHeader_2.54mm:PinHeader_1x08_P2.54mm_Vertical, symbol Connector:Conn_01x08_Pin
- added J8: Solar_panel_connector, Connector_PinHeader_2.54mm:PinHeader_1x02_P2.54mm_Vertical, symbol Connector:Conn_01x02_Socket
- added J9: AVR-ISP-6, Connector_PinHeader_2.54mm:PinHeader_2x03_P2.54mm_Vertical, symbol Connector:AVR-ISP-6
- added Q2: SSM3J371R, Package_TO_SOT_SMD:SOT-23-3, symbol Simulation_SPICE:PMOS
- added R17: 2k2, Resistor_SMD:R_0805_2012Metric_Pad1.20x1.40mm_HandSolder, symbol Device:R
- added R18, R19, R20, R21: 4k7, Resistor_SMD:R_0805_2012Metric_Pad1.20x1.40mm_HandSolder, symbol Device:R
- added U7: SN74LS07N, Package_DIP:DIP-14_W7.62mm, symbol 74xx:SN74LS07N
- C1, C11, C12, C2, C4, C8, C9: footprint Capacitor_THT:C_Disc_D3.4mm_W2.1mm_P2.50mm -> Capacitor_SMD:C_0805_2012Metric_Pad1.18x1.45mm_HandSolder
- C13, C20, C6, C7: footprint Capacitor_THT:CP_Radial_D5.0mm_P2.50mm -> Capacitor_SMD:C_0805_2012Metric_Pad1.18x1.45mm_HandSolder
- C18, C19: footprint Capacitor_THT:CP_Radial_D5.0mm_P2.50mm -> Capacitor_SMD:C_1206_3216Metric_Pad1.33x1.80mm_HandSolder
- D2: footprint Diode_THT:D_A-405_P10.16mm_Horizontal -> Diode_THT:D_DO-35_SOD27_P7.62mm_Horizontal
- J6: footprint (none) -> Connector_PinHeader_2.54mm:PinHeader_1x02_P2.54mm_Vertical
- L3: footprint Inductor_SMD:L_Wuerth_WE-PD2-Typ-L -> inductor_footprint:WE-PD2_1054
- Q1: value PMOS -> SSM3J371R
- U2: footprint (none) -> Package_SO:TSSOP-8_4.4x3mm_P0.65mm
Connections:
- net +3.3VDc: now also Q1.2 (S), U1.27 (AVCC), C21.1, J5.2 (Pin_2), J7.2 (Pin_2), R19.1, R20.1, R21.1; no longer Q1.3 (S)
- net CS_0: now also J5.7 (Pin_7)
- net GND: now also BT1.2 (-), C21.2, C22.2, J5.3 (Pin_3), J7.1 (Pin_1), J8.1 (Pin_1), J9.6 (GND), U7.11, U7.13, U7.7 (GND)
- net LiPo_Battery: now also BT1.1 (+), D4.1 (K), Q2.2 (S); no longer R13.1
- net MISO: now also J5.5 (Pin_5), U7.1
- net MOSI: now also J5.6 (Pin_6), R19.2, U7.4
- net RST: now also R21.2, U7.8
- net SCK: now also J5.4 (Pin_4), R20.2, U7.6
- net Solar_panel: now also J8.2 (Pin_2)
- net at Q1.1 (G): now also R10.1; no longer R11.1
- net PD2: now reaches U1.11 (PD2)
- net PD2: now also J7.5 (Pin_5)
- net PD3: now reaches U1.12 (PD3)
- net PD3: now also J7.4 (Pin_4)
- net PD4: now reaches U1.13 (PD4)
- net PD4: now also J7.3 (Pin_3)
- net CS_BLVL: now reaches U1.22 (PC3)
- net CS_BLVL: now also R17.2
- net PA5: now reaches U1.32 (PA5)
- net PA5: now also J7.7 (Pin_7)
- net PA4: now reaches U1.33 (PA4)
- net PA4: now also J7.8 (Pin_8)
- net PB0: now reaches U1.40 (PB0)
- net PB0: now also J7.6 (Pin_6)
- new net: Q1.3 (D), R11.1
- new net: Q2.1 (G), R17.1
- new net: Q2.3 (D), R13.1
- new net +5VDc: R18.1
- new net +5VDc_ISP: C22.1, D4.2 (A), J9.2 (VCC), U7.14 (VCC)
- new net MISO_5V: J9.1 (MISO), R18.2, U7.2
- new net MOSI_5V: J9.4 (MOSI), U7.3
- new net RST_5V: J9.5 (~{RST}), U7.9
- new net SCK_5V: J9.3 (SCK), U7.5
- no-connect marks 1 -> 16
Other:
- note added: "Empty pins for later prototyping"
- note added: "ICSP prog. header with logic leven converter"
- note removed: "ICSP header"
- company: (none) -> Axel Söderberg
- moved on the sheet: C1, C10, C11, C12, C13, C14, C15, C16, C17, C18, C19, C2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
