File: KiCad_projekti/Elektroniikkapaja-vastaanotin/Elektroniikkapaja-vastaanotin.kicad_sch (KiCad schematic)
At the start: 29 parts, among them J1 USB_A, J2 Conn_Coaxial, U1 ATmega328PB-A, U2 MICRF220AYQS, U3 FT230XS, U4 MCP1700x-330xxTO, Y1 Crystal

Commit message: nyt on valmista levyä
Parts:
- removed J1: USB_A, symbol Connector:USB_A
- removed L1: L, symbol Device:L
- added C12, C14, C18, C20, C21: 100nF, Capacitor_SMD:C_0805_2012Metric_Pad1.18x1.45mm_HandSolder, symbol Device:C
- added C13: 10uF, Capacitor_SMD:C_0805_2012Metric_Pad1.18x1.45mm_HandSolder, symbol Device:C
- added C15, C16: 22pF, Capacitor_SMD:C_0805_2012Metric_Pad1.18x1.45mm_HandSolder, symbol Device:C
- added C17: 4.7uF, Capacitor_SMD:C_1206_3216Metric_Pad1.33x1.80mm_HandSolder, symbol Device:C
- added C19: 1.2pF, Capacitor_SMD:C_0805_2012Metric_Pad1.18x1.45mm_HandSolder, symbol Device:C
- added D3, D4, D5: LED, LED_SMD:LED_0805_2012Metric_Pad1.15x1.40mm_HandSolder, symbol Device:LED
- added H1, H2, H3, H4: MountingHole, MountingHole:MountingHole_2.2mm_M2, symbol Mechanical:MountingHole
- added J1: USB_B, Connector_USB:USB_B_Lumberg_2411_02_Horizontal, symbol Connector:USB_B
- added J3: Conn_01x04_Pin, Connector_JST:JST_SH_SM04B-SRSS-TB_1x04-1MP_P1.00mm_Horizontal, symbol Connector:Conn_01x04_Pin
- added J4: AVR-ISP-6, Connector_PinHeader_2.54mm:PinHeader_2x03_P2.54mm_Vertical, symbol Connector:AVR-ISP-6
- added J5: Conn_01x04_Pin, Connector_PinHeader_2.54mm:PinHeader_1x04_P2.54mm_Vertical, symbol Connector:Conn_01x04_Pin
- added J6: Conn_01x06_Pin, Connector_PinHeader_2.54mm:PinHeader_1x06_P2.54mm_Vertical, symbol Connector:Conn_01x06_Pin
- added J7: Conn_01x08_Pin, Connector_PinHeader_2.54mm:PinHeader_1x08_P2.54mm_Vertical, symbol Connector:Conn_01x08_Pin
- added L2: 39nH, Capacitor_SMD:C_0805_2012Metric_Pad1.18x1.45mm_HandSolder, symbol Device:L
- added R10, R11, R8, R9: 4k7, Resistor_SMD:R_0805_2012Metric_Pad1.20x1.40mm_HandSolder, symbol Device:R
- added R12: 10k, Resistor_SMD:R_0805_2012Metric_Pad1.20x1.40mm_HandSolder, symbol Device:R
- added R13: 150r, Resistor_SMD:R_0805_2012Metric, symbol Device:R
- added R7: 330r, Resistor_SMD:R_0805_2012Metric_Pad1.20x1.40mm_HandSolder, symbol Device:R
- added SW_reset1: SW_Push, Button_Switch_SMD:SW_SPST_TL3305A, symbol Switch:SW_Push
- added U5: TL072, Package_SO:SOIC-8_3.9x4.9mm_P1.27mm, symbol Amplifier_Operational:TL072
- added U6: SN74LS07N, Package_DIP:DIP-14_W7.62mm, symbol 74xx:SN74LS07N
- added Y2: Crystal 16MHz, Crystal:Crystal_HC49-U_Vertical, symbol Device:Crystal
- C1, C2: value C -> 47pF; footprint (none) -> Capacitor_SMD:C_0805_2012Metric_Pad1.18x1.45mm_HandSolder
- C10, C11, C4, C5: value C -> 100nF; footprint (none) -> Capacitor_SMD:C_0805_2012Metric_Pad1.18x1.45mm_HandSolder
- C3: value C -> 4.7uF; footprint (none) -> Capacitor_SMD:C_1206_3216Metric_Pad1.33x1.80mm_HandSolder
- C6, C7: value C -> 1uF; footprint (none) -> Capacitor_SMD:C_0805_2012Metric_Pad1.18x1.45mm_HandSolder
- C8, C9: value C -> 10pF; footprint (none) -> Capacitor_SMD:C_0805_2012Metric_Pad1.18x1.45mm_HandSolder
- D1, D2: footprint (none) -> LED_SMD:LED_0805_2012Metric_Pad1.15x1.40mm_HandSolder
- J2: footprint (none) -> Connector_Coaxial:SMA_Amphenol_901-143_Horizontal
- JP1: renamed from JP2; footprint (none) -> Jumper:SolderJumper-3_P1.3mm_Open_RoundedPad1.0x1.5mm_NumberLabels
- JP2: renamed from JP1; footprint (none) -> Jumper:SolderJumper-3_P1.3mm_Open_RoundedPad1.0x1.5mm_NumberLabels
- R1, R2: value R -> 560R; footprint (none) -> Resistor_SMD:R_0805_2012Metric_Pad1.20x1.40mm_HandSolder
- R3, R4: value R -> 27R; footprint (none) -> Resistor_SMD:R_0805_2012Metric_Pad1.20x1.40mm_HandSolder
- R5: value R -> 150r; footprint (none) -> Resistor_SMD:R_0805_2012Metric_Pad1.20x1.40mm_HandSolder
- R6: value R -> 100r; footprint (none) -> Resistor_SMD:R_0805_2012Metric_Pad1.20x1.40mm_HandSolder
- Y1: value Crystal -> 13.52313MHz; footprint (none) -> Crystal:Crystal_SMD_HC49-SD_HandSoldering
Connections:
- net +3.3VDc: now also C10.1, U1.18 (AVCC), U1.4 (VCC), C12.1, C13.1, C14.1, J3.2 (Pin_2), J5.2 (Pin_2), J6.3 (Pin_3), J7.2 (Pin_2), R10.1, R11.1, R12.1, R9.1, U5.8 (V+)
- net +5VDc: now also C21.1, J1.1 (VBUS), J4.2 (VCC), R8.1, U6.14 (VCC)
- net GND: now also C10.2, C12.2, C13.2, C14.2, C15.1, C16.1, C17.2, C18.1, C20.2, C21.2, D3.1 (K), D4.1 (K), D5.1 (K), J1.4 (GND), J3.1 (Pin_1), J4.6 (GND), J5.1 (Pin_1), J6.1 (Pin_1), J7.1 (Pin_1), L2.1, R7.1, SW_reset1.1, U5.4 (V-), U6.11, U6.13, U6.7 (GND)
- net RSSI: now also U5.5 (+)
- net RST: now also R11.2, R12.2, SW_reset1.2, U6.8
- net Rx: now also U3.1 (TXD), J6.4 (Pin_4); no longer R5.2
- net Tx: now also U3.4 (RXD), J6.5 (Pin_5); no longer R6.2
- net at J2.1 (In): now also C19.2; no longer C10.1
- net at U2.3 (ANT): now also C19.1, L2.2; no longer C10.2
- net at R5.1: now also U5.1, U5.2 (-); no longer U3.1 (TXD)
- net at C5.1, U3.10 (3V3OUT), U3.3 (VCCIO): now also U3.11 (~{RESET})
- net RTS: now reaches C4.1, U3.2 (~{RTS})
- net RTS: now also J6.6 (Pin_6)
- net at R6.1: now also U5.6 (-), U5.7; no longer U3.4 (RXD)
- net at C2.1, R4.1: now also J1.3 (D+)
- net ASK_demodulated: now reaches U2.10 (DO)
- net ASK_demodulated: now also U1.11 (PD7), U5.3 (+)
- net at U2.12 (CTH): now also C18.2
- net at U2.13 (CAGC): now also C17.1
- net at C1.1, R3.1: now also J1.2 (D-)
- net PD3: now reaches U1.1 (PD3)
- net PD3: now also J7.4 (Pin_4)
- net PB1: now reaches U1.13 (PB1)
- net PB1: now also J7.8 (Pin_8)
- net int_led: now reaches U1.14 (PB2)
- net int_led: now also R13.1
- net MOSI_3.3V: now reaches U1.15 (PB3)
- net MOSI_3.3V: now also R9.2, U6.4
- net MISO_3.3V: now reaches U1.16 (PB4)
- net MISO_3.3V: now also U6.1
- net SCK_3.3V: now reaches U1.17 (PB5)
- net SCK_3.3V: now also R10.2, U6.6
- net PD4: now reaches U1.2 (PD4)
- net PD4: now also J7.3 (Pin_3)
- net PC1: now reaches U1.24 (PC1)
- net PC1: now also J7.7 (Pin_7)
- net PC2: now reaches U1.25 (PC2)
- net PC2: now also J7.6 (Pin_6)
- net PC3: now reaches U1.26 (PC3)
- net PC3: now also J7.5 (Pin_5)
- net SDA: now reaches U1.27 (PC4)
- net SDA: now also J3.3 (Pin_3), J5.3 (Pin_3)
- net SCL: now reaches U1.28 (PC5)
- net SCL: now also J3.4 (Pin_4), J5.4 (Pin_4)
- net at U1.7 (XTAL1/PB6): now also C15.2, Y2.2
- net at U1.8 (XTAL2/PB7): now also C16.2, Y2.1
- new net: C20.1, J1.5 (Shield), R7.2
- new net: D5.2 (A), R13.2
- new net: D4.2 (A), R6.2
- new net: D3.2 (A), R5.2
- new net MISO_5V: J4.1 (MISO), R8.2, U6.2
- new net MOSI_5V: J4.4 (MOSI), U6.3
- new net RST_5V: J4.5 (~{RST}), U6.9
- new net SCK_5V: J4.3 (SCK), U6.5
- no-connect marks 0 -> 15
Other:
- note added: "Buffered Rx & RSSI leds"
- note added: "ICSP prog. header with logic level converter"
- note added: "OLED SSD1306 I2C"
- note added: "UART header"
- note added: "Unused pins for later prototyping"
- company: (none) -> Axel Söderberg
- moved on the sheet: C2, C3, C4, C5, C6, C7, D1, D2, J2, R1, R3, U1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
